File: matrix.sch (KiCad schematic (older format))
At the start: 358 parts

Commit message: Simplify layout, remove LEDs and alps support, and start revising footprint positioning.
Parts:
- removed D102, D103, D104, D105, D106, D107, D109, D110, D114, D14, D15, D16, D31, D32, D33, D34, D49, D50, D51, D64, D66, D79, D80, D83, D88, D89, D98: SOD-323, Diodes_SMD:D_SOD-123, symbol Device:D_Small
- removed MX_BACK2, MX_BACK3, MX_LSHIFT3, MX_NUM1, MX_NUM10, MX_NUM11, MX_NUM12, MX_NUM13, MX_NUM14, MX_NUM15, MX_NUM16, MX_NUM17, MX_NUM18, MX_NUM19, MX_NUM2, MX_NUM20, MX_NUM21, MX_NUM22, MX_NUM23, MX_NUM24, MX_NUM3, MX_NUM4, MX_NUM5, MX_NUM6, MX_NUM7, MX_NUM8, MX_NUM9, MX_RSHIFT3, MX_\2: MX-1U, MX_Alps_Hybrid:MX-1U, symbol MX_Alps_Hybrids:MX-1U
- removed MX_CLOCK2: MX-1.25U, MX_Alps_Hybrid:MX-1.25U-FLIPPED, symbol MX_Alps_Hybrids:MX-1.25U
- removed MX_LALT2, MX_LCTRL2: MX-1.5U, MX_Alps_Hybrid:MX-1.5U-FLIPPED, symbol MX_Alps_Hybrids:MX-1.5U
- removed MX_LGUI2: MX-1U, MX_Alps_Hybrid:MX-1U-FLIPPED, symbol MX_Alps_Hybrids:MX-1.5U
- removed MX_LSHIFT2: MX-1.25U, MX_Alps_Hybrid:MX-1.25U, symbol MX_Alps_Hybrids:MX-2.25U
- removed MX_NUM_EX1, MX_NUM_EX2, MX_NUM_EX3: MX-2U, MX_Alps_Hybrid:MX-2U-ReversedStabilizers, symbol MX_Alps_Hybrids:MX-1U
- removed MX_RALT2, MX_RCTRL2: MX-1.5U, MX_Alps_Hybrid:MX-1.5U, symbol MX_Alps_Hybrids:MX-1.5U
- removed MX_RETURN2: MX-ISO, MX_Alps_Hybrid:MX-ISO-ReversedStabilizers, symbol MX_Alps_Hybrids:MX-2.25U
- removed MX_RGUI2: MX-1U, MX_Alps_Hybrid:MX-1U, symbol MX_Alps_Hybrids:MX-1.5U
- removed MX_RSHIFT2: MX-1.75U, MX_Alps_Hybrid:MX-1.75U, symbol MX_Alps_Hybrids:MX-1U
- removed MX_SP2: MX-7U, MX_Alps_Hybrid:MX-7U-ReversedStabilizers, symbol MX_Alps_Hybrids:MX-7U
- removed R1, R10, R100, R101, R102, R103, R104, R105, R106, R107, R108, R109, R11, R110, R111, R112, R113, R114, R12, R13, R14, R15, R16, R17, R18, R19, R2, R20, R21, R22, R23, R24, R25, R26, R27, R28, R29, R3, R30, R31, R32, R33, R34, R35, R36, R37, R38, R39, R4, R40, R41, R42, R43, R44, R45, R46, R47, R48, R49, R5, R50, R51, R52, R53, R54, R55, R56, R57, R58, R59, R6, R60, R61, R62, R63, R64, R65, R66, R67, R68, R69, R7, R70, R71, R72, R73, R74, R75, R76, R77, R78, R79, R8, R80, R81, R82, R83, R84, R85, R86, R87, R88, R89, R9, R90, R91, R92, R93, R94, R95, R96, R97, R98, R99: 1k, Resistors_SMD:R_0603, symbol Device:R_Small
- MX_#0_1, MX_#1, MX_#2, MX_#3, MX_#4, MX_#5, MX_#6, MX_#7, MX_#8, MX_#9, MX_'1, MX_,1, MX_-1, MX_.1, MX_/1, MX_;1, MX_=1, MX_A1, MX_B1, MX_C1, MX_D1, MX_DEL1, MX_DN1, MX_E1, MX_END1, MX_ESC1, MX_F1, MX_FN1, MX_FN10, MX_FN11, MX_FN12, MX_FN2, MX_FN3, MX_FN4, MX_FN5, MX_FN6, MX_FN7, MX_FN8, MX_FN9, MX_G1, MX_H1, MX_HOME1, MX_I1, MX_INS1, MX_J1, MX_K1, MX_L1, MX_LFT1, MX_M1, MX_N1, MX_O1, MX_P1, MX_PAUSE1, MX_PGDN1, MX_PGUP1, MX_PRINT1, MX_Q1, MX_R1, MX_RT1, MX_S1, MX_SLOCK1, MX_T1, MX_U1, MX_UP1, MX_V1, MX_W1, MX_X1, MX_Y1, MX_Z1, MX_[1, MX_]1, MX_`1: footprint MX_Alps_Hybrid:MX-1U -> Button_Switch_Keyboard:SW_Cherry_MX1A_1.00u_PCB; symbol MX_Alps_Hybrids:MX-1U -> Voyager104-rescue:MX-1U-MX_Alps_Hybrids
- MX_BACK1: footprint MX_Alps_Hybrid:MX-2U -> Button_Switch_Keyboard:SW_Cherry_MX1A_2.00u_PCB; symbol MX_Alps_Hybrids:MX-2U -> Voyager104-rescue:MX-2U-MX_Alps_Hybrids
- MX_CLOCK1: footprint MX_Alps_Hybrid:MX-1.75U -> Button_Switch_Keyboard:SW_Cherry_MX1A_1.75u_PCB; symbol MX_Alps_Hybrids:MX-1.75U -> Voyager104-rescue:MX-1.75U-MX_Alps_Hybrids
- MX_LALT1, MX_LGUI1, MX_RALT1: footprint MX_Alps_Hybrid:MX-1.25U -> Button_Switch_Keyboard:SW_Cherry_MX1A_1.25u_PCB; symbol MX_Alps_Hybrids:MX-1.25U -> Voyager104-rescue:MX-1.25U-MX_Alps_Hybrids
- MX_LCTRL1: footprint MX_Alps_Hybrid:MX-1.25U -> Button_Switch_Keyboard:SW_Cherry_MX1A_1.25u_PCB; symbol MX_Alps_Hybrids:MX-1U -> Voyager104-rescue:MX-1U-MX_Alps_Hybrids
- MX_LSHIFT1, MX_RETURN1: footprint MX_Alps_Hybrid:MX-2.25U -> Button_Switch_Keyboard:SW_Cherry_MX1A_2.25u_PCB; symbol MX_Alps_Hybrids:MX-2.25U -> Voyager104-rescue:MX-2.25U-MX_Alps_Hybrids
- MX_RCTRL1, MX_RMENU1: footprint MX_Alps_Hybrid:MX-1.25U-FLIPPED -> Button_Switch_Keyboard:SW_Cherry_MX1A_1.25u_PCB; symbol MX_Alps_Hybrids:MX-1U -> Voyager104-rescue:MX-1U-MX_Alps_Hybrids
- MX_RGUI1: footprint MX_Alps_Hybrid:MX-1.25U-FLIPPED -> Button_Switch_Keyboard:SW_Cherry_MX1A_1.25u_PCB; symbol MX_Alps_Hybrids:MX-1.25U -> Voyager104-rescue:MX-1.25U-MX_Alps_Hybrids
- MX_RSHIFT1: footprint MX_Alps_Hybrid:MX-2.75U -> Button_Switch_Keyboard:SW_Cherry_MX1A_2.75u_PCB; symbol MX_Alps_Hybrids:MX-1U -> Voyager104-rescue:MX-1U-MX_Alps_Hybrids
- MX_SP1: footprint MX_Alps_Hybrid:MX-6.25U-ReversedStabilizers -> Button_Switch_Keyboard:SW_Cherry_MX1A_6.25u_PCB; symbol MX_Alps_Hybrids:MX-6.25U -> Voyager104-rescue:MX-6.25U-MX_Alps_Hybrids
- MX_TAB1, MX_\1: footprint MX_Alps_Hybrid:MX-1.5U -> Button_Switch_Keyboard:SW_Cherry_MX1A_1.50u_PCB; symbol MX_Alps_Hybrids:MX-1.5U -> Voyager104-rescue:MX-1.5U-MX_Alps_Hybrids
Connections:
- net labels removed: +5V, COL17, COL18, COL19, COL20, LEDGND
- wire segments 1142 -> 436
