File: Voyager104.kicad_pcb (KiCad board)
At the start: 2 copper layers, 425.4 x 123.4 mm, 383 parts, among them J1 AVR-ISP-6, Q1 DSS60601MZ4-13, SW1 SW_Push, U1 AT90USB1286-AU, U2 PRTR5V0U2X, Y1 16MHz

Commit message: Simplify layout, remove LEDs and alps support, and start revising footprint positioning.
Parts:
- removed D102, D103, D104, D105, D106, D107, D109, D110, D114, D14, D15, D16, D31, D32, D33, D34, D49, D50, D51, D64, D66, D79, D80, D83, D88, D89, D98: SOD-323, Diodes_SMD:D_SOD-123
- removed G***: LOGO, locallib:ai-ring-6mm
- removed G***: LOGO, locallib:ai-ring-6mm-FancyAss
- removed G***: LOGO, locallib:ai-ring-6mm-FancyAss-Mask
- removed MX_BACK2, MX_BACK3, MX_LSHIFT3, MX_NUM1, MX_NUM10, MX_NUM11, MX_NUM12, MX_NUM13, MX_NUM14, MX_NUM15, MX_NUM16, MX_NUM17, MX_NUM18, MX_NUM19, MX_NUM2, MX_NUM20, MX_NUM21, MX_NUM22, MX_NUM23, MX_NUM24, MX_NUM3, MX_NUM4, MX_NUM5, MX_NUM6, MX_NUM7, MX_NUM8, MX_NUM9, MX_RGUI2, MX_RSHIFT3, MX_\2: MX-1U, MX_Alps_Hybrid:MX-1U
- removed MX_CLOCK2: MX-1.25U, MX_Alps_Hybrid:MX-1.25U-FLIPPED
- removed MX_LALT2, MX_LCTRL2: MX-1.5U, MX_Alps_Hybrid:MX-1.5U-FLIPPED
- removed MX_LGUI2: MX-1U, MX_Alps_Hybrid:MX-1U-FLIPPED
- removed MX_LSHIFT2: MX-1.25U, MX_Alps_Hybrid:MX-1.25U
- removed MX_NUM_EX1, MX_NUM_EX2, MX_NUM_EX3: MX-2U, MX_Alps_Hybrid:MX-2U-ReversedStabilizers
- removed MX_RALT2, MX_RCTRL2: MX-1.5U, MX_Alps_Hybrid:MX-1.5U
- removed MX_RETURN2: MX-ISO, MX_Alps_Hybrid:MX-ISO-ReversedStabilizers
- removed MX_RSHIFT2: MX-1.75U, MX_Alps_Hybrid:MX-1.75U
- removed MX_SP2: MX-7U, MX_Alps_Hybrid:MX-7U-ReversedStabilizers
- removed Q1: DSS60601MZ4-13, TO_SOT_Packages_SMD:SOT-223-3_TabPin2
- removed R1, R10, R100, R101, R102, R103, R104, R105, R106, R107, R108, R109, R11, R110, R111, R112, R113, R114, R12, R13, R14, R15, R16, R17, R18, R19, R2, R20, R21, R22, R23, R24, R25, R26, R27, R28, R29, R3, R30, R31, R32, R33, R34, R35, R36, R37, R38, R39, R4, R40, R41, R42, R43, R44, R45, R46, R47, R48, R49, R5, R50, R51, R52, R53, R54, R55, R56, R57, R58, R59, R6, R60, R61, R62, R63, R64, R65, R66, R67, R68, R69, R7, R70, R71, R72, R73, R74, R75, R76, R77, R78, R79, R8, R80, R81, R82, R83, R84, R85, R86, R87, R88, R89, R9, R90, R91, R92, R93, R94, R95, R96, R97, R98, R99: 1k, Resistors_SMD:R_0603
- removed RC5: 1.5k, Resistors_SMD:R_0603
- MX_#0_1, MX_#1, MX_#2, MX_#3, MX_#4, MX_#5, MX_#6, MX_#7, MX_#8, MX_#9, MX_'1, MX_,1, MX_-1, MX_.1, MX_/1, MX_;1, MX_=1, MX_A1, MX_B1, MX_C1, MX_D1, MX_DEL1, MX_DN1, MX_E1, MX_END1, MX_ESC1, MX_F1, MX_FN1, MX_FN10, MX_FN11, MX_FN12, MX_FN2, MX_FN3, MX_FN4, MX_FN5, MX_FN6, MX_FN7, MX_FN8, MX_FN9, MX_G1, MX_H1, MX_HOME1, MX_I1, MX_INS1, MX_J1, MX_K1, MX_L1, MX_LFT1, MX_M1, MX_N1, MX_O1, MX_P1, MX_PAUSE1, MX_PGDN1, MX_PGUP1, MX_PRINT1, MX_Q1, MX_R1, MX_RT1, MX_S1, MX_SLOCK1, MX_T1, MX_U1, MX_UP1, MX_V1, MX_W1, MX_X1, MX_Y1, MX_Z1, MX_[1, MX_]1, MX_`1: footprint MX_Alps_Hybrid:MX-1U -> Button_Switch_Keyboard:SW_Cherry_MX1A_1.00u_PCB
- MX_BACK1: footprint MX_Alps_Hybrid:MX-2U -> Button_Switch_Keyboard:SW_Cherry_MX1A_2.00u_PCB
- MX_CLOCK1: footprint MX_Alps_Hybrid:MX-1.75U -> Button_Switch_Keyboard:SW_Cherry_MX1A_1.75u_PCB
- MX_LALT1, MX_LCTRL1, MX_LGUI1, MX_RALT1: footprint MX_Alps_Hybrid:MX-1.25U -> Button_Switch_Keyboard:SW_Cherry_MX1A_1.25u_PCB
- MX_LSHIFT1, MX_RETURN1: footprint MX_Alps_Hybrid:MX-2.25U -> Button_Switch_Keyboard:SW_Cherry_MX1A_2.25u_PCB
- MX_RCTRL1, MX_RGUI1, MX_RMENU1: footprint MX_Alps_Hybrid:MX-1.25U-FLIPPED -> Button_Switch_Keyboard:SW_Cherry_MX1A_1.25u_PCB
- MX_RSHIFT1: footprint MX_Alps_Hybrid:MX-2.75U -> Button_Switch_Keyboard:SW_Cherry_MX1A_2.75u_PCB
- MX_SP1: footprint MX_Alps_Hybrid:MX-6.25U-ReversedStabilizers -> Button_Switch_Keyboard:SW_Cherry_MX1A_6.25u_PCB
- MX_TAB1, MX_\1: footprint MX_Alps_Hybrid:MX-1.5U -> Button_Switch_Keyboard:SW_Cherry_MX1A_1.50u_PCB
Connections:
- U1 pad 1: Net-(U1-Pad1) -> (no net)
- U1 pad 10: Net-(U1-Pad10) -> (no net)
- U1 pad 14: Net-(U1-Pad14) -> (no net)
- U1 pad 15: Net-(U1-Pad15) -> (no net)
- U1 pad 16: Net-(U1-Pad16) -> (no net)
- U1 pad 17: Net-(RC5-Pad1) -> (no net)
- U1 pad 18: Net-(U1-Pad18) -> (no net)
- U1 pad 19: Net-(U1-Pad19) -> (no net)
- U1 pad 2: Net-(U1-Pad2) -> (no net)
- U1 pad 25: Net-(U1-Pad25) -> (no net)
- U1 pad 26: Net-(U1-Pad26) -> (no net)
- U1 pad 27: Net-(U1-Pad27) -> (no net)
- U1 pad 28: Net-(U1-Pad28) -> (no net)
- U1 pad 29: Net-(U1-Pad29) -> (no net)
- U1 pad 30: Net-(U1-Pad30) -> (no net)
- U1 pad 33: COL20 -> (no net)
- U1 pad 34: COL19 -> (no net)
- U1 pad 35: COL18 -> (no net)
- U1 pad 36: COL17 -> (no net)
- U1 pad 44: Net-(U1-Pad44) -> (no net)
- U1 pad 62: Net-(U1-Pad62) -> (no net)
- U1 pad 9: Net-(U1-Pad9) -> (no net)
- USB1 pad 3: Net-(USB1-Pad3) -> (no net)
- USB1 pad 9: Net-(USB1-Pad9) -> (no net)
Routing:
- net +5V: track 2935.1 -> 160.3 mm, vias 13 -> 9
- net LEDGND: track 2285.2 -> 426.5 mm, vias 18 -> 7
- net COL6: track 708.8 -> 0.00 mm
- net COL7: track 690.8 -> 0.00 mm
- net COL5: track 621.4 -> 0.00 mm
- net COL8: track 574.4 -> 0.00 mm
- net COL4: track 564.4 -> 0.00 mm, vias 1 -> 0
- net ROW2: track 519.3 -> 4.28 mm, vias 4 -> 1
- net COL3: track 504.2 -> 0.00 mm, vias 2 -> 0
- net COL9: track 479.7 -> 0.00 mm
- net COL2: track 474.3 -> 0.00 mm, vias 2 -> 0
- net COL0: track 470.7 -> 0.00 mm
- net ROW1: track 539.0 -> 111.6 mm, vias 5 -> 3
- net COL1: track 423.9 -> 0.00 mm
- net COL10: track 408.0 -> 0.00 mm, vias 1 -> 0
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Other:
- board size 425.4 x 123.4 mm -> 429.4 x 130.6 mm
- board text removed: "Voyager104 PCB Rev 1.0 20190216"

Commit message: Revise pcb futher.
Parts:
- moved MX_ESC1 5.93 mm to (43.0, 35.9)
- moved MX_FN10 5.43 mm to (271.6, 36.8)
- moved MX_FN2 5.43 mm to (100.2, 36.8)
- moved MX_FN3 5.43 mm to (119.2, 36.8)
- moved MX_FN4 5.43 mm to (138.3, 36.8)
- moved MX_FN6 5.43 mm to (185.9, 36.8)
- moved MX_FN7 5.43 mm to (205.0, 36.8)
- moved MX_FN8 5.43 mm to (224.0, 36.8)
- moved MX_FN9 5.43 mm to (252.6, 36.8)
- moved MX_FN1 5.43 mm to (81.1, 36.8)
- moved MX_FN11 5.43 mm to (290.7, 36.8)
- moved MX_FN12 5.43 mm to (309.7, 36.8)
- moved MX_FN5 5.43 mm to (166.9, 36.8)
- moved MX_=1 4.62 mm to (271.6, 63.0)
- moved MX_BACK1 4.62 mm to (300.2, 63.0)
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Other:
- board size 429.4 x 130.6 mm -> 435.1 x 130.6 mm

Commit message: Initial revision for as yet unnamed project.
Parts:
- removed J1: AVR-ISP-6, random-keyboard-parts:Reset_Pretty-Mask
- removed RC6, RC7: 5k1, Resistors_SMD:R_0603
- removed USB1: HRO-TYPE-C-31-M-12, Type-C:HRO-TYPE-C-31-M-12-Assembly
- added J2: USB_B_Mini, Connectors_JST:JST_PH_S5B-PH-SM4-TB_05x2.00mm_Angled, F.Cu at (315.7, 52.6)
- moved D67 38.6 mm to (44.4, 124.9)
- moved D87 35.4 mm to (154.0, 143.9)
- moved U2 32.9 mm to (314.5, 65.7), turned to 90 degrees
- moved D84 26.1 mm to (34.9, 143.9)
- moved D85 26.1 mm to (58.7, 143.9)
- moved D86 26.1 mm to (82.5, 143.9)
- moved D52 23.8 mm to (39.7, 105.8)
- moved D35 23.8 mm to (37.3, 86.8)
- moved D17 23.8 mm to (32.5, 67.7)
- moved D18 23.8 mm to (51.6, 67.7)
- moved D53 23.8 mm to (65.8, 105.8)
- moved D36 23.8 mm to (61.1, 86.8)
- moved D68 23.8 mm to (75.4, 124.9)
- moved D19 23.8 mm to (70.6, 67.7)
- moved D54 23.8 mm to (84.9, 105.8)
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Connections:
- net RESET renamed Net-(RC3-Pad2)
- U1 pad 11: SCK -> (no net)
- U1 pad 12: MOSI -> (no net)
- U1 pad 13: MISO -> (no net)
Routing:
- net ROW2: track 4.28 -> 439.1 mm, vias 1 -> 0
- net LEDGND: track 426.5 -> 0.00 mm, vias 7 -> 0
- net COL0: track 0.00 -> 417.5 mm, vias 0 -> 1
- net COL2: track 0.00 -> 379.1 mm, vias 0 -> 1
- net COL1: track 0.00 -> 357.4 mm, vias 0 -> 1
- net ROW5: track 44.9 -> 384.8 mm
- net COL3: track 0.00 -> 334.7 mm, vias 0 -> 1
- net ROW1: track 111.6 -> 439.7 mm, vias 3 -> 2
- net COL4: track 0.00 -> 313.1 mm, vias 0 -> 1
- net ROW0: track 149.6 -> 459.3 mm
- net COL6: track 0.00 -> 305.6 mm, vias 0 -> 1
- net COL5: track 0.00 -> 297.3 mm, vias 0 -> 1
- net ROW4: track 62.9 -> 335.1 mm
- net COL7: track 0.00 -> 266.9 mm, vias 0 -> 1
- net ROW3: track 80.7 -> 330.6 mm
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Other:
- board size 435.1 x 130.6 mm -> 349.1 x 124.8 mm
- board text added: "Nova MX 0 by Faux Learning Machine Adapted from ai03's Voyager104"
- board text removed: "104"
- board text removed: "VOYAGER"
- board text removed: "kb.ai03.me"
