File: Voyager104.sch (KiCad schematic (older format))
At the start: 22 parts, among them J1 AVR-ISP-6, Q1 DSS60601MZ4-13, SW1 SW_Push, U1 AT90USB1286-AU, U2 PRTR5V0U2X, Y1 16MHz

Commit message: Simplify layout, remove LEDs and alps support, and start revising footprint positioning.
Parts:
- removed Q1: DSS60601MZ4-13, TO_SOT_Packages_SMD:SOT-223-3_TabPin2, symbol Device:Q_NPN_BCE
- removed RC5: 1.5k, Resistors_SMD:R_0603, symbol Device:R_Small
- U1: symbol MCU_Microchip_AVR:AT90USB1286-MU -> Voyager104-rescue:AT90USB1286-MU-MCU_Microchip_AVR
- USB1: symbol Type-C:HRO-TYPE-C-31-M-12 -> Voyager104-rescue:HRO-TYPE-C-31-M-12-Type-C
Connections:
- net labels removed: COL17, COL18, COL19, COL20, LEDGND
- wire segments 84 -> 82
- no-connect marks 3 -> 24
Changed lines of the file:
@@
 D+
-$Comp
-L Device:Q_NPN_BCE Q1
-U 1 1 5A4CAD6E
-P 6425 4875
-F 0 "Q1" H 6625 4925 50  0000 L CNN
-F 1 "DSS60601MZ4-13" H 6625 4825 50  0000 L CNN
-F 2 "TO_SOT_Packages_SMD:SOT-223-3_TabPin2" H 6625 4975 50  0001 C CNN
-F 3 "" H 6425 4875 50  0001 C CNN
-	1    6425 4875
-	1    0    0    -1
-$EndComp
-Text GLabel 6525 4675 1    60   Input ~ 0
-LEDGND
-$Comp
-L power:GND #PWR02
-U 1 1 5A4CB170
-P 6525 5075
-F 0 "#PWR02" H 6525 4825 50  0001 C CNN
-F 1 "GND" H 6525 4925 50  0000 C CNN
-F 2 "" H 6525 5075 50  0001 C CNN
-F 3 "" H 6525 5075 50  0001 C CNN
-	1    6525 5075
-	1    0    0    -1
-$EndComp
-$Comp
-L Device:R_Small RC5
-U 1 1 5A4CB690
-P 5875 4875
-F 0 "RC5" V 5950 4875 50  0000 L CNN
-F 1 "1.5k" V 5950 4700 50  0000 L CNN
-F 2 "Resistors_SMD:R_0603" H 5875 4875 50  0001 C CNN
-F 3 "" H 5875 4875 50  0001 C CNN
-	1    5875 4875
-	0    -1   -1   0
-$EndComp
 $Comp
 L power:VCC #PWR03
@@
 	3175 1400 3125 1400
 Wire Wire Line
-	5975 4875 6225 4875
-Wire Wire Line
 	3525 4575 3925 4575
 Wire Wire Line
@@
 Connection ~ 1650 5375
 Wire Wire Line
-	5775 4875 5125 4875
-Wire Wire Line
 	2925 850  3100 850
 Wire Wire Line
@@
 MISO
 $Comp
-L Type-C:HRO-TYPE-C-31-M-12 USB1
+L Voyager104-rescue:HRO-TYPE-C-31-M-12-Type-C USB1
 U 1 1 5BE083A1
 P 1350 1450
@@
 Connection ~ 4525 2975
 $Comp
-L MCU_Microchip_AVR:AT90USB1286-MU U1
+L Voyager104-rescue:AT90USB1286-MU-MCU_Microchip_AVR U1
 U 1 1 5B32E6E2
 P 4525 4975
@@
 Connection ~ 4000 2975
 Connection ~ 3725 3275
-Text GLabel 5125 5175 2    50   Input ~ 0
-COL17
-Text GLabel 5125 5075 2    50   Input ~ 0
-COL18
-Text GLabel 3925 5175 0    50   Input ~ 0
-COL19
-Text GLabel 3925 5075 0    50   Input ~ 0
-COL20
+NoConn ~ 3925 5075
+NoConn ~ 3925 5175
+NoConn ~ 3925 5375
+NoConn ~ 3925 5475
+NoConn ~ 3925 5575
+NoConn ~ 3925 5675
+NoConn ~ 3925 5775
+NoConn ~ 5125 4175
+NoConn ~ 5125 3975
+NoConn ~ 5125 4575
+NoConn ~ 5125 5075
+NoConn ~ 5125 5175
+NoConn ~ 5125 5975
+NoConn ~ 5125 6075
+NoConn ~ 5125 6175
+NoConn ~ 5125 6275
+NoConn ~ 5125 6375
+NoConn ~ 5125 6475
+NoConn ~ 5125 4675
+NoConn ~ 5125 4775
+NoConn ~ 5125 4875
 $EndSCHEMATC

Commit message: Initial revision for as yet unnamed project.
Parts:
- removed J1: AVR-ISP-6, random-keyboard-parts:Reset_Pretty-Mask, symbol Connector:AVR-ISP-6
- removed RC6, RC7: 5k1, Resistors_SMD:R_0603, symbol Device:R_Small
- removed USB1: HRO-TYPE-C-31-M-12, Type-C:HRO-TYPE-C-31-M-12-Assembly, symbol Voyager104-rescue:HRO-TYPE-C-31-M-12-Type-C
- added J2: USB_B_Mini, Connectors_JST:JST_PH_S5B-PH-SM4-TB_05x2.00mm_Angled, symbol faux:USB_B_Mini
Connections:
- net GND: now also J2.2 (Shield)
- net VCC: now also J2.1 (VBUS)
- net at RC1.2, U2.3 (IO2): now also J2.3 (D+)
- net at RC2.1, U2.2 (IO1): now also J2.4 (D-)
- net MISO: no longer names the net of U1.13 (PB3)
- net MOSI: no longer names the net of U1.12 (PB2)
- net RESET: no longer names the net of RC3.2, SW1.2, U1.20 (~RESET)
- net SCK: no longer names the net of U1.11 (PB1)
- no-connect marks 24 -> 26
Other:
- moved on the sheet: F1, RC1, RC2, U2
